Commit message: Updated score functions

File: src/bulletwalker/assets/urdfs/models/model.urdf (robot description, URDF)
Before this commit: robot passive_walker, 7 links, 6 joints
Links:
- removed link left_foot_custom_frame
- removed link right_foot_custom_frame
- link left_foot: mass 0.5 -> 3.0; geometry collision mesh filename=../../meshes/foot_2.obj scale=0.3 0.3 0.3; visual mesh filename=../../meshes/foot_2.obj scale=0.3 0.3 0.3
- link right_foot: geometry collision mesh filename=../../meshes/foot_2.obj scale=0.3 0.3 0.3; visual mesh filename=../../meshes/foot_2.obj scale=0.3 0.3 0.3
Joints:
- removed joint left_foot_to_left_foot_custom_frame
- removed joint right_foot_to_right_foot_custom_frame
- joint left_hip: origin xyz=0.0 -0.4 0.0 rpy=0.0 0.0 0.0 -> xyz=0.0 -0.47 0.0 rpy=0.0 0.0 0.0
- joint right_hip: limit lower=-0.5235987755982988 upper=0.5235987755982988 effort=3.4028235e+38 velocity=3.4028235e+38 -> lower=-0.5235987755982988 upper=0.5235987755982988 effort=1e+9 velocity=1e+9; origin xyz=0.0 0.4 0.0 rpy=0.0 0.0 0.0 -> xyz=0.0 0.47 0.0 rpy=0.0 0.0 0.0
